Commit message: Wire Vention rail into URDF and SRDF
URDF (picknik_007_rail.xacro):
- Include vention_mo_lm_039_2295_macro.xacro
- Insert linear_actuator_ + pedestal + 45° robot adapter + mount_link
  between world and the arm; reparent the UR arm onto
  linear_actuator_robot_mount_link instead of world
- Add rail_ip xacro arg (default 192.168.7.2)

SRDF (picknik_007_rail.srdf):
- Add planning groups: linear_actuator (chain on the rail) and
  linear_actuator_and_manipulator (combined for whole-body planning)
- Move virtual_joint child_link from base_link -> linear_actuator_base_link
  (the rail base is what's now fixed to the world frame)
- Add hand-picked disable_collisions for rail-chain adjacency. The full
  collision matrix should be regenerated via MoveIt Setup Assistant once
  the URDF is final.

Also fixed a sed regression that incorrectly renamed the upstream
picknik_accessories camera adapter filename.

File: src/picknik_007_rail_mock/description/picknik_007_rail.xacro (robot description, xacro)
@@ -3,6 +3,9 @@
   <!-- robot name parameter -->
   <xacro:arg name="name" default="ur"/>
-  <!-- import main macro -->
+  <!-- import main macros -->
   <xacro:include filename="$(find ur_description)/urdf/ur_macro.xacro"/>
+  <xacro:include filename="$(find vention_description)/urdf/vention_mo_lm_039_2295_macro.xacro"/>
+  <!-- IP address of the Vention MachineMotion 2 controller for the linear rail -->
+  <xacro:arg name="rail_ip" default="192.168.7.2"/>
   <!-- possible 'ur_type' values: ur3, ur3e, ur5, ur5e, ur10, ur10e, ur16e, ur20, ur30 -->
   <!-- the default value should raise an error in case this was called without defining the type -->
@@ -49,9 +52,71 @@
   <!-- create link fixed to the "world" -->
   <link name="world" />
+  <!-- Linear rail: Vention MachineMotion 2 (MO-LM-039-2295). The macro creates
+       linear_actuator_base_link (mounted on world) and linear_actuator_carriage_link
+       (the moving carriage), connected by the prismatic linear_actuator_carriage_joint. -->
+  <xacro:linear_actuator
+    parent="world"
+    prefix="linear_actuator_"
+    ip_address="$(arg rail_ip)"
+    use_fake_hardware="$(arg use_fake_hardware)"
+  >
+    <origin xyz="0 0 0" rpy="0 0 0"/>
+  </xacro:linear_actuator>
+  <!-- Pedestal cylinder on the rail carriage. -->
+  <link name="linear_actuator_pedestal_link">
+    <visual>
+      <geometry><cylinder length="0.61" radius="0.105"/></geometry>
+      <origin xyz="0 0 0.305"/>
+    </visual>
+    <collision>
+      <geometry><cylinder length="0.61" radius="0.105"/></geometry>
+      <origin xyz="0 0 0.305"/>
+    </collision>
+    <inertial>
+      <mass value="10"/>
+      <inertia ixx="1.0" ixy="0.0" ixz="0.0" iyy="1.0" iyz="0.0" izz="1.0"/>
+    </inertial>
+  </link>
+  <joint name="linear_actuator_pedestal_joint" type="fixed">
+    <parent link="linear_actuator_carriage_link"/>
+    <child link="linear_actuator_pedestal_link"/>
+    <origin rpy="0 0 ${pi}" xyz="0.09 0 0.045"/>
+  </joint>
+  <!-- 45-degree robot adapter plate (McMaster 6333N39). -->
+  <link name="linear_actuator_robot_adapter_link">
+    <visual>
+      <geometry>
+        <mesh filename="package://vention_description/meshes/visual/6333N39_45deg_Robot_Base.dae"/>
+      </geometry>
+      <origin xyz="0 0 0"/>
+    </visual>
+    <collision>
+      <geometry>
+        <mesh filename="package://vention_description/meshes/collision/6333N39_45deg_Robot_Base.stl"/>
+      </geometry>
+      <origin xyz="0 0 0"/>
+    </collision>
+    <inertial>
+      <mass value="10"/>
+      <inertia ixx="1.0" ixy="0.0" ixz="0.0" iyy="1.0" iyz="0.0" izz="1.0"/>
+    </inertial>
+  </link>
+  <joint name="linear_actuator_robot_adapter_joint" type="fixed">
+    <parent link="linear_actuator_pedestal_link"/>
+    <child link="linear_actuator_robot_adapter_link"/>
+    <origin rpy="0 0 0" xyz="0 0 0.6096"/>
+  </joint>
+  <!-- Robot mount frame: 45° pitch around Y, where the arm base attaches. -->
+  <link name="linear_actuator_robot_mount_link"/>
+  <joint name="linear_actuator_robot_mount_joint" type="fixed">
+    <parent link="linear_actuator_robot_adapter_link"/>
+    <child link="linear_actuator_robot_mount_link"/>
+    <origin rpy="0 ${pi/4} 0" xyz="0.048 0 0.134"/>
+  </joint>
   <!-- arm -->
   <xacro:ur_robot
           name="$(arg name)"
           tf_prefix="$(arg tf_prefix)"
-          parent="world"
+          parent="linear_actuator_robot_mount_link"
           joint_limits_parameters_file="$(arg joint_limit_parameters_file)"
           kinematics_parameters_file="$(arg kinematics_params)"

Commit message: Restore rail support frame + carriage adapter; rotate arm 180° on mount
I had over-trimmed vention_description by excluding nasa_frame.dae and
nasa_carriage_adapter.dae. The picknik_007 cell uses the same support
frame and carriage adapter as the original NASA cell, so the meshes
need to be present (visually and to anchor the rail at the correct
height above the floor). Restored both files (~50 MB combined).

URDF (picknik_007_rail.xacro):
- Add linear_actuator_frame_link with the support-frame mesh; world is
  now fixed to the frame, not directly to the rail base
- Reparent the linear_actuator macro from world onto the frame_link
  with the offset that was on linear_actuator_base_joint in the source
  (xyz=0.2475 -0.0675 0.275)
- Insert linear_actuator_carriage_adapter_link between carriage_link
  and the pedestal; collision boxes match the source URDF
- Rotate the arm 180° around Z at the mount-link attach (origin rpy
  0 0 pi). Without this the UR base faced the back of the
  electronics-side wall.

SRDF:
- virtual_joint child_link: linear_actuator_base_link -> linear_actuator_frame_link
- Add disable_collisions for the frame link and carriage_adapter_link
  with the obvious adjacent/never pairs. Still hand-picked; full matrix
  should be regenerated via MoveIt Setup Assistant before final use.

File: src/picknik_007_rail_mock/description/picknik_007_rail.xacro (robot description, xacro)
@@ -51,4 +51,10 @@
        UR but skip the Vention driver (e.g., while it's being debugged). -->
   <xacro:arg name="rail_use_fake_hardware" default="$(arg use_fake_hardware)"/>
+  <!-- Same idea for the Robotiq gripper. The real driver activates as part of
+       the same ros2_control_node as the UR, but its on_activate() runs before
+       the UR has pushed the rs485 URScript, so it times out. Force the gripper
+       to mock_components/GenericSystem here while we sort that out; flip back
+       to "false" once rs485 over /tmp/ttyUR is verified. -->
+  <xacro:arg name="gripper_use_fake_hardware" default="$(arg use_fake_hardware)"/>
   <!-- initial position for simulations (Fake Hardware, Gazebo, Ignition) -->
   <xacro:arg name="initial_positions_file" default="$(find ur_description)/config/initial_positions.yaml"/>
@@ -57,16 +63,76 @@
   <!-- create link fixed to the "world" -->
   <link name="world" />
-  <!-- Linear rail: Vention MachineMotion 2 (MO-LM-039-2295). The macro creates
-       linear_actuator_base_link (mounted on world) and linear_actuator_carriage_link
-       (the moving carriage), connected by the prismatic linear_actuator_carriage_joint. -->
+  <!-- Frame that the rail sits on. The visual mesh (nasa_frame.dae) was the
+       support structure built for the original NASA cell; the picknik_007 cell
+       reuses the same frame. Collision is approximated with two boxes (the
+       base profile and the electronics-side wall). -->
+  <link name="linear_actuator_frame_link">
+    <visual>
+      <geometry>
+        <mesh filename="package://vention_description/meshes/visual/nasa_frame.dae"/>
+      </geometry>
+      <origin xyz="0 0 0"/>
+    </visual>
+    <collision>
+      <geometry><box size="0.82 2.7 0.365"/></geometry>
+      <origin xyz="0.365 0 0.183"/>
+    </collision>
+    <collision>
+      <geometry><box size="0.2 2.7 0.865"/></geometry>
+      <origin xyz="0.660 0 0.433"/>
+    </collision>
+    <inertial>
+      <mass value="100"/>
+      <inertia ixx="1.0" ixy="0.0" ixz="0.0" iyy="1.0" iyz="0.0" izz="1.0"/>
+    </inertial>
+  </link>
+  <joint name="linear_actuator_frame_joint" type="fixed">
+    <parent link="world"/>
+    <child link="linear_actuator_frame_link"/>
+    <origin rpy="0 0 0" xyz="0 0 0"/>
+  </joint>
+  <!-- Linear rail: Vention MachineMotion 2 (MO-LM-039-2295). Mounts on the
+       frame at the offset measured for the picknik_007/NASA cell. The macro
+       creates linear_actuator_{base,carriage,motor}_link plus the prismatic
+       linear_actuator_carriage_joint. -->
   <xacro:linear_actuator
-    parent="world"
+    parent="linear_actuator_frame_link"
     prefix="linear_actuator_"
     ip_address="$(arg rail_ip)"
     use_fake_hardware="$(arg rail_use_fake_hardware)"
   >
-    <origin xyz="0 0 0" rpy="0 0 0"/>
+    <origin xyz="0.2475 -0.0675 0.275" rpy="0 0 0"/>
   </xacro:linear_actuator>
-  <!-- Pedestal cylinder on the rail carriage. -->
+  <!-- Carriage adapter plate that the pedestal bolts to. -->
+  <link name="linear_actuator_carriage_adapter_link">
+    <visual>
+      <geometry>
+        <mesh filename="package://vention_description/meshes/visual/nasa_carriage_adapter.dae"/>
+      </geometry>
+      <origin xyz="0 0 0"/>
+    </visual>
+    <collision>
+      <geometry><box size="0.410 0.4 0.045"/></geometry>
+      <origin xyz="0.093 0 0.0225"/>
+    </collision>
+    <collision>
+      <geometry><box size="0.275 0.088 0.230"/></geometry>
+      <origin xyz="-0.135 -0.158 0.115"/>
+    </collision>
+    <collision>
+      <geometry><box size="0.1 0.4 0.150"/></geometry>
+      <origin xyz="-0.150 -0.4 0.075"/>
+    </collision>
+    <inertial>
+      <mass value="100"/>
+      <inertia ixx="1.0" ixy="0.0" ixz="0.0" iyy="1.0" iyz="0.0" izz="1.0"/>
+    </inertial>
+  </link>
+  <joint name="linear_actuator_carriage_adapter_joint" type="fixed">
+    <parent link="linear_actuator_carriage_link"/>
+    <child link="linear_actuator_carriage_adapter_link"/>
+    <origin rpy="0 0 0" xyz="0 0 0"/>
+  </joint>
+  <!-- Pedestal cylinder on the carriage adapter. -->
   <link name="linear_actuator_pedestal_link">
     <visual>
@@ -84,5 +150,5 @@
   </link>
   <joint name="linear_actuator_pedestal_joint" type="fixed">
-    <parent link="linear_actuator_carriage_link"/>
+    <parent link="linear_actuator_carriage_adapter_link"/>
     <child link="linear_actuator_pedestal_link"/>
     <origin rpy="0 0 ${pi}" xyz="0.09 0 0.045"/>
@@ -157,5 +223,7 @@
           trajectory_port="$(arg trajectory_port)"
   >
-    <origin xyz="0 0 0" rpy="0 0 0" />          <!-- position robot in the world -->
+    <!-- 180° yaw so the UR base faces the opposite side of the 45° mount.
+         (Without this, the arm faces the back of the rail's electronics wall.) -->
+    <origin xyz="0 0 0" rpy="0 0 ${pi}"/>
   </xacro:ur_robot>
   <!-- Gripper, UR adapter, and realsense camera -->
@@ -198,5 +266,5 @@
     prefix="$(arg tf_prefix)"
     parent="gripper_mount_link"
-    use_fake_hardware="$(arg use_fake_hardware)"
+    use_fake_hardware="$(arg gripper_use_fake_hardware)"
     sim_ignition="false"
     com_port="$(arg tool_device_name)"
